File: vibrovario2.kicad_pcb (KiCad board)
At the start: 4 copper layers, 33.8 x 46 mm, 86 parts, among them J1 Battery, J2 Micro USB, J3 FPC24(0.5MM), M1 Vibration_Motor, Q1 CJ2301, Q2 S8050, Q3 AO3400A, SW1 BTN2, SW2 BTN1, SW3 BTN3, SW4 BTN4, U1 SR2HARU, U2 RT908033, U3 TP4054, U4 ESP32-S3, U5 USBLC6-2P6, U6 BMA423, Y1 32.768KHz, Y2 40MHz

Commit message: Add files via upload
Parts:
- added C22: 100nF, Capacitor_SMD:C_0402_1005Metric, F.Cu at (80.5, 89.5)
- added C23: 1uF, Capacitor_SMD:C_0402_1005Metric, F.Cu at (80.5, 91.0)
- added U5: BMP390, vibrovario2:BMP390_LGA-10, F.Cu at (82.5, 89.5)
Connections:
- U4 pad 51: unconnected-(U4-GPIO45-Pad51) -> BMP390_PWR
Routing:
- net BMP390_PWR: track 0.00 -> 7.05 mm
- net SDA: track 22.1 -> 28.7 mm
- net SCL: track 26.3 -> 32.6 mm
Changed lines of the file:
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@@
   (net 61 "USB_D-")
   (net 62 "USB_D+")
-  (net 63 "unconnected-(U4-GPIO45-Pad51)")
+  (net 63 "BMP390_PWR")
   (net 64 "unconnected-(U4-MTMS{slash}JTAG{slash}GPIO42-Pad48)")
   (net 65 "unconnected-(U4-MTDI{slash}JTAG{slash}GPIO41-Pad47)")
@@
       (net 55 "Net-(U4-U0RXD{slash}PROG{slash}GPIO44)") (pinfunction "U0RXD/PROG/GPIO44") (pintype "bidirectional"))
     (pad "51" smd roundrect (at -0.6 -3.4375 270) (size 0.2 0.875) (layers "F.Cu" "F.Paste" "F.Mask") (roundrect_rratio 0.25)
-      (net 63 "unconnected-(U4-GPIO45-Pad51)") (pinfunction "GPIO45") (pintype "bidirectional+no_connect"))
+      (net 63 "BMP390_PWR") (pinfunction "GPIO45") (pintype "bidirectional"))
     (pad "52" smd roundrect (at -1 -3.4375 270) (size 0.2 0.875) (layers "F.Cu" "F.Paste" "F.Mask") (roundrect_rratio 0.25)
       (net 60 "unconnected-(U4-GPIO46-Pad52)") (pinfunction "GPIO46") (pintype "bidirectional+no_connect"))
@@
     )
   )
+  (footprint "vibrovario2:BMP390_LGA-10" (layer "F.Cu")
+    (at 82.5 89.5)
+    (descr "BMP390 Barometric Pressure Sensor, LGA-10, 2.0x2.0x0.75mm")
+    (tags "BMP390 pressure sensor LGA-10")
+    (property "Sheetfile" "vibrovario2.kicad_sch")
+    (property "Sheetname" "")
+    (property "LCSC" "C496091")
+    (property "MPN" "BMP390")
+    (property "Manufacturer" "Bosch Sensortec")
+    (property "Description" "Digital Pressure Sensor")
+    (attr smd)
+    (fp_text reference "U5" (at 0 -2) (layer "F.SilkS")
+      (effects (font (size 0.8 0.8) (thickness 0.12)))
+      (tstamp bmp390_ref)
+    )
+    (fp_text value "BMP390" (at 0 2) (layer "F.Fab")
+      (effects (font (size 0.8 0.8) (thickness 0.12)))
+      (tstamp bmp390_val)
+    )
+    (fp_text user "${REFERENCE}" (at 0 0) (layer "F.Fab")
+      (effects (font (size 0.5 0.5) (thickness 0.08)))
+    )
+    (fp_line (start -1.1 -1.1) (end 1.1 -1.1) (stroke (width 0.05) (type solid)) (layer "F.CrtYd"))
+    (fp_line (start 1.1 -1.1) (end 1.1 1.1) (stroke (width 0.05) (type solid)) (layer "F.CrtYd"))
+    (fp_line (start 1.1 1.1) (end -1.1 1.1) (stroke (width 0.05) (type solid)) (layer "F.CrtYd"))
+    (fp_line (start -1.1 1.1) (end -1.1 -1.1) (stroke (width 0.05) (type solid)) (layer "F.CrtYd"))
+    (fp_line (start -1 -1) (end -1 1) (stroke (width 0.1) (type solid)) (layer "F.Fab"))
+    (fp_line (start -1 1) (end 1 1) (stroke (width 0.1) (type solid)) (layer "F.Fab"))
+    (fp_line (start 1 1) (end 1 -1) (stroke (width 0.1) (type solid)) (layer "F.Fab"))
+    (fp_line (start 1 -1) (end -1 -1) (stroke (width 0.1) (type solid)) (layer "F.Fab"))
+    (fp_line (start -1 -0.6) (end -0.6 -1) (stroke (width 0.1) (type solid)) (layer "F.Fab"))
+    (fp_line (start -1.05 -1.05) (end 1.05 -1.05) (stroke (width 0.12) (type solid)) (layer "F.SilkS"))
+    (fp_line (start 1.05 -1.05) (end 1.05 1.05) (stroke (width 0.12) (type solid)) (layer "F.SilkS"))
+    (fp_line (start 1.05 1.05) (end -1.05 1.05) (stroke (width 0.12) (type solid)) (layer "F.SilkS"))
+    (fp_line (start -1.05 1.05) (end -1.05 -1.05) (stroke (width 0.12) (type solid)) (layer "F.SilkS"))
+    (fp_circle (center -0.7 -0.7) (end -0.6 -0.7) (stroke (width 0.15) (type solid)) (fill none) (layer "F.SilkS"))
+    (pad "1" smd rect (at -0.75 -0.5) (size 0.3 0.4) (layers "F.Cu" "F.Paste" "F.Mask")
+      (net 1 "GND") (pinfunction "GND") (pintype "power_in") (tstamp p1))
+    (pad "2" smd rect (at -0.75 0) (size 0.3 0.4) (layers "F.Cu" "F.Paste" "F.Mask")
+      (net 2 "+3V3") (pinfunction "VDDIO") (pintype "power_in") (tstamp p2))
+    (pad "3" smd rect (at -0.75 0.5) (size 0.3 0.4) (layers "F.Cu" "F.Paste" "F.Mask")
+      (net 1 "GND") (pinfunction "SDO") (pintype "input") (tstamp p3))
+    (pad "4" smd rect (at -0.75 0.9) (size 0.3 0.25) (layers "F.Cu" "F.Paste" "F.Mask")
+      (net 0 "") (pinfunction "INT2") (pintype "output") (tstamp p4))
+    (pad "5" smd rect (at -0.45 0.9) (size 0.3 0.25) (layers "F.Cu" "F.Paste" "F.Mask")
+      (net 63 "BMP390_PWR") (pinfunction "VDD") (pintype "power_in") (tstamp p5))
+    (pad "6" smd rect (at 0.45 0.9) (size 0.3 0.25) (layers "F.Cu" "F.Paste" "F.Mask")
+      (net 0 "") (pinfunction "INT1") (pintype "output") (tstamp p6))
+    (pad "7" smd rect (at 0.75 0.5) (size 0.3 0.4) (layers "F.Cu" "F.Paste" "F.Mask")
+      (net 20 "SCL") (pinfunction "SCL") (pintype "input") (tstamp p7))
+    (pad "8" smd rect (at 0.75 0) (size 0.3 0.4) (layers "F.Cu" "F.Paste" "F.Mask")
+      (net 19 "SDA") (pinfunction "SDA") (pintype "bidirectional") (tstamp p8))
+    (pad "9" smd rect (at 0.75 -0.5) (size 0.3 0.4) (layers "F.Cu" "F.Paste" "F.Mask")
+      (net 2 "+3V3") (pinfunction "CSB") (pintype "input") (tstamp p9))
+    (pad "10" smd rect (at 0.75 -0.9) (size 0.3 0.25) (layers "F.Cu" "F.Paste" "F.Mask")
+      (net 1 "GND") (pinfunction "GND") (pintype "power_in") (tstamp p10))
+  )
+  (footprint "Capacitor_SMD:C_0402_1005Metric" (layer "F.Cu")
+    (at 80.5 89.5)
+    (descr "Capacitor SMD 0402 (1005 Metric)")
+    (tags "capacitor")
+    (property "Sheetfile" "vibrovario2.kicad_sch")
+    (property "Sheetname" "")
+    (property "LCSC" "C1525")
+    (property "MPN" "CL05B104JB5NNNC")
+    (property "Description" "100nF 0402 capacitor")
+    (attr smd)
+    (fp_text reference "C22" (at 0 -1.16) (layer "F.SilkS") hide
+      (effects (font (size 1 1) (thickness 0.15)))
+    )
+    (fp_text value "100nF" (at 0 1.16) (layer "F.Fab")
+      (effects (font (size 1 1) (thickness 0.15)))
+    )
+    (fp_line (start -0.91 -0.46) (end 0.91 -0.46) (stroke (width 0.05) (type solid)) (layer "F.CrtYd"))
+    (fp_line (start -0.91 0.46) (end -0.91 -0.46) (stroke (width 0.05) (type solid)) (layer "F.CrtYd"))
+    (fp_line (start 0.91 -0.46) (end 0.91 0.46) (stroke (width 0.05) (type solid)) (layer "F.CrtYd"))
+    (fp_line (start 0.91 0.46) (end -0.91 0.46) (stroke (width 0.05) (type solid)) (layer "F.CrtYd"))
+    (fp_line (start -0.5 -0.25) (end 0.5 -0.25) (stroke (width 0.1) (type solid)) (layer "F.Fab"))
+    (fp_line (start -0.5 0.25) (end -0.5 -0.25) (stroke (width 0.1) (type solid)) (layer "F.Fab"))
+    (fp_line (start 0.5 -0.25) (end 0.5 0.25) (stroke (width 0.1) (type solid)) (layer "F.Fab"))
+    (fp_line (start 0.5 0.25) (end -0.5 0.25) (stroke (width 0.1) (type solid)) (layer "F.Fab"))
+    (pad "1" smd roundrect (at -0.48 0) (size 0.56 0.62) (layers "F.Cu" "F.Paste" "F.Mask") (roundrect_rratio 0.25)
+      (net 63 "BMP390_PWR") (pintype "passive"))
+    (pad "2" smd roundrect (at 0.48 0) (size 0.56 0.62) (layers "F.Cu" "F.Paste" "F.Mask") (roundrect_rratio 0.25)
+      (net 1 "GND") (pintype "passive"))
+  )
+  (footprint "Capacitor_SMD:C_0402_1005Metric" (layer "F.Cu")
+    (at 80.5 91.0)
+    (descr "Capacitor SMD 0402 (1005 Metric)")
+    (tags "capacitor")
+    (property "Sheetfile" "vibrovario2.kicad_sch")
+    (property "Sheetname" "")
+    (property "LCSC" "C52923")
+    (property "MPN" "CL05A105KA5NQNC")
+    (property "Description" "1uF 0402 capacitor")
+    (attr smd)
+    (fp_text reference "C23" (at 0 -1.16) (layer "F.SilkS") hide
+      (effects (font (size 1 1) (thickness 0.15)))
+    )
+    (fp_text value "1uF" (at 0 1.16) (layer "F.Fab")
+      (effects (font (size 1 1) (thickness 0.15)))
+    )
+    (fp_line (start -0.91 -0.46) (end 0.91 -0.46) (stroke (width 0.05) (type solid)) (layer "F.CrtYd"))
+    (fp_line (start -0.91 0.46) (end -0.91 -0.46) (stroke (width 0.05) (type solid)) (layer "F.CrtYd"))
+    (fp_line (start 0.91 -0.46) (end 0.91 0.46) (stroke (width 0.05) (type solid)) (layer "F.CrtYd"))
+    (fp_line (start 0.91 0.46) (end -0.91 0.46) (stroke (width 0.05) (type solid)) (layer "F.CrtYd"))
+    (fp_line (start -0.5 -0.25) (end 0.5 -0.25) (stroke (width 0.1) (type solid)) (layer "F.Fab"))
+    (fp_line (start -0.5 0.25) (end -0.5 -0.25) (stroke (width 0.1) (type solid)) (layer "F.Fab"))
+    (fp_line (start 0.5 -0.25) (end 0.5 0.25) (stroke (width 0.1) (type solid)) (layer "F.Fab"))
+    (fp_line (start 0.5 0.25) (end -0.5 0.25) (stroke (width 0.1) (type solid)) (layer "F.Fab"))
+    (pad "1" smd roundrect (at -0.48 0) (size 0.56 0.62) (layers "F.Cu" "F.Paste" "F.Mask") (roundrect_rratio 0.25)
+      (net 63 "BMP390_PWR") (pintype "passive"))
+    (pad "2" smd roundrect (at 0.48 0) (size 0.56 0.62) (layers "F.Cu" "F.Paste" "F.Mask") (roundrect_rratio 0.25)
+      (net 1 "GND") (pintype "passive"))
+  )
+  (segment (start 85.52 86.51) (end 82.05 89.98) (width 0.2) (layer "F.Cu") (net 63) (tstamp seg_bmp_pwr_1))
+  (segment (start 82.05 89.98) (end 82.05 90.4) (width 0.2) (layer "F.Cu") (net 63) (tstamp seg_bmp_pwr_2))
+  (segment (start 81.78 89.5) (end 81.75 89.5) (width 0.2) (layer "F.Cu") (net 63) (tstamp seg_bmp_pwr_3))
+  (segment (start 81.75 89.5) (end 82.05 89.8) (width 0.2) (layer "F.Cu") (net 63) (tstamp seg_bmp_pwr_4))
+  (segment (start 83.25 90.4) (end 82.05 89.98) (width 0.2) (layer "F.Cu") (net 63) (tstamp seg_bmp_pwr_5))
+  (segment (start 83.25 89.0) (end 84.0 89.0) (width 0.2) (layer "F.Cu") (net 20) (tstamp seg_scl_1))
+  (segment (start 84.0 89.0) (end 89.5575 89.0) (width 0.2) (layer "F.Cu") (net 20) (tstamp seg_scl_2))
+  (segment (start 83.25 89.5) (end 84.5 89.5) (width 0.2) (layer "F.Cu") (net 19) (tstamp seg_sda_1))
+  (segment (start 84.5 89.5) (end 89.5575 87.71) (width 0.2) (layer "F.Cu") (net 19) (tstamp seg_sda_2))
 )
