File: vibrovario2.kicad_sch (KiCad schematic)
At the start: 82 parts, among them J1 Battery, J2 Micro USB, J3 FPC24(0.5MM), M1 Vibration_Motor, Q1 CJ2301, Q2 S8050, Q3 AO3400A, SW1 BTN2, SW2 BTN1, SW3 BTN3, SW4 BTN4, U1 SR2HARU, U2 RT908033, U3 TP4054, U4 ESP32-S3, U5 USBLC6-2P6, U6 BMA423, Y1 32.768KHz, Y2 40MHz

Commit message: Add files via upload
Parts:
- added C22: 100nF, Capacitor_SMD:C_0402_1005Metric, symbol Device:C
- added C23: 1uF, Capacitor_SMD:C_0402_1005Metric, symbol Device:C
- added U5: BMP390, vibrovario2:BMP390_LGA-10, symbol BMP390:BMP390
Connections:
- net 40M_N: now also C23.2
Other:
- company: SQFMI -> VibroVario Project
- title: Watchy -> VibroVario2
